File: hardware/kicad_session1/lri_s1/lri_s1.kicad_sch (KiCad schematic)
At the start: 21 parts, among them J1 USB_C_Receptacle_USB2.0_16P, Q2 NMOS, SW1 MJTP1230, SW2 MJTP1230, U1 STM32F042F6Px, U2 LP5912-3.3DRV

Commit message: Updated onboarding project
Parts:
- added C10, C14: 2.2u, symbol Device:C_Small
- added C11, C12, C13, C8, C9: 100n, symbol Device:C_Small
- added D3: RED, symbol Device:LED_Small
- added J2, J3: PY1, symbol Connector:Screw_Terminal_01x02
- added Q2: NMOS, symbol Simulation_SPICE:NMOS
- added Q3: CSD17318Q2, Package_SON:Texas_DQK, symbol Transistor_FET:CSD17313Q2
- added R10, R8: 100, symbol Device:R_Small
- added R7: 1k, symbol Device:R_Small
- added R9: 10k, symbol Device:R_Small
- added U3: ICM-20602, Package_LGA:LGA-16_3x3mm_P0.5mm_LayoutBorder3x5y, symbol Sensor_Motion:ICM-20602
- added U4: BMP280, Package_LGA:Bosch_LGA-8_2x2.5mm_P0.65mm_ClockwisePinNumbering, symbol Sensor_Pressure:BMP280
- U1: value STM32F042F6Px -> STM32F042F6P6
- renumbered Q2 to Q1
Connections:
- net +3V3: now also C10.2, C12.2, C13.2, C14.2, C8.2, C9.2, U3.1 (VDDIO), U3.16 (VDD), U4.6 (VDDIO), U4.8 (VDD)
- net GND: now also C10.1, C11.2, C12.1, C13.1, C14.1, C8.1, C9.1, D3.1 (K), J3.2 (Pin_2), Q3.4 (S), Q3.7 (S), R9.1, U3.10 (GND), U3.11 (GND), U3.12 (GND), U3.13 (GND), U3.15 (GND), U3.8 (FSYNC), U3.9 (GND), U4.1 (GND), U4.7 (GND)
- net MCU_LED: now also U1.6 (PA0); no longer U1.9 (PA3)
- net VBUS: now also R7.2
- net BMP_~{CS}: now reaches U1.10 (PA4)
- net BMP_~{CS}: now also U4.2 (CSB)
- net SPI1_MOSI: now reaches U1.11 (PA5)
- net SPI1_MOSI: now also U3.3 (SDA/SDI), U4.3 (SDI)
- net SPI1_MISO: now reaches U1.12 (PA6)
- net SPI1_MISO: now also U3.4 (SAO/SD0), U4.4 (SCK)
- net SPI1_SCK: now reaches U1.13 (PA7)
- net SPI1_SCK: now also U3.2 (SCL/SPC), U4.5 (SDO)
- net MCU_PY1: now reaches U1.7 (PA1)
- net USB_PD+ renamed USB_D+
- net USB_PD- renamed USB_D-
- new net: Q3.3 (G), R8.1, R9.2
- new net: D3.2 (A), Q2.3 (S)
- new net: J2.2 (Pin_2), R10.1
- new net: Q3.1 (D), Q3.2 (D), Q3.5 (D), Q3.6 (D), Q3.8 (D), R10.2
- new net: C11.1, U3.14 (REGOUT)
- new net: Q2.1 (D), R7.1
- new net +12V: J2.1 (Pin_1), J3.1 (Pin_1)
- new net ICM_~{CS}: U1.9 (PA3), U3.5 (~{CS})
- new net MCU_PYRO: Q2.2 (G), R8.2
- no-connect marks 14 -> 10
Other:
- note added: "120 mA STM32, 4.2 uA BMP, 2.79 mA ICM"
- note added: "ACCELEROMETER + GYROSCOPE"
- note added: "BAROMETER"
- note added: "CAN CUT LATER IF SHORT ON TIME"
- note added: "HEAT LOSSES: P = (V_IN – V_OUT) * I_LOAD P = (5.0 V - 3.3 V) * 123 mA = 210 mW MAX"
- note added: "MOUNTING HOLES"
- note added: "NEGLECT TO ADD ESD PROTECTION FOR SIMPLICITY PURPOSES"
- note added: "PYROS"
- note added: "SPI"
- note added: "STM32 INTRO FC"
- note added: "USB"
- note added: "VDD + VDDIO TIED TOGETHER TO HAVE ICM I/O BE 3V3 USE X7R CAPS SEE DATASHEET 4.8 FOR SPI CONNECTIONS"
- note removed: "STM32 W/ USB-C PD"
- moved on the sheet: C6, C7, D1, D2, Q1, R4, R5, R6, U2

Commit message: Resolved ERC errors.
Parts:
- added H1, H2, H3, H4: MountingHole, symbol Mechanical:MountingHole
- added R11, R13: 100, symbol Device:R_Small
- added R12, R14: 10k, symbol Device:R_Small
Connections:
- net GND: now also R12.1, R14.1
- net MCU_LED: now also R11.2; no longer Q1.2 (G)
- net MCU_PY1: now also R8.2, R13.2
- net MCU_PYRO: no longer names the net of Q2.2 (G)
- net MCU_PYRO: now also R13.1, R14.2; no longer R8.2
- new net: Q1.2 (G), R11.1, R12.2
- no-connect marks 10 -> 11
Other:
- note added: "[1] STM32 INTRO FC"
- note removed: "STM32 INTRO FC"
